File: PowerSupply.kicad_pcb (KiCad board)
At the start: 2 copper layers, 30 x 26 mm, 19 parts, among them Q1 Q_PMOS_GDS, U1 LM25085

Commit message: Second commit
Parts:
- moved R1 7.80 mm to (106.0, 82.5), turned to -90 degrees
- moved C3 4.91 mm to (104.0, 82.5), turned to -90 degrees
Routing:
- net Vin: track 25.6 -> 38.4 mm
- net Net-(R1-Pad2): track 7.57 -> 17.4 mm
- net Net-(C3-Pad2): track 7.11 -> 3.67 mm
Other:
- board text added: "Switching node of the PFET must be kept small to avoid radiations, but must be big to dissipate power"

Commit message: Sch update 08/21
Parts:
- removed C7, C8: 22uF, Capacitor_SMD:C_1206_3216Metric_Pad1.33x1.80mm_HandSolder
- removed R6: 9K1, Resistor_SMD:R_0805_2012Metric_Pad1.20x1.40mm_HandSolder
- removed R7: 270, Resistor_SMD:R_0805_2012Metric_Pad1.20x1.40mm_HandSolder
- C1: value 33uF -> 10uF; footprint Capacitor_SMD:C_1206_3216Metric_Pad1.33x1.80mm_HandSolder -> Capacitor_SMD:C_1210_3225Metric_Pad1.33x2.70mm_HandSolder
- C2: footprint Capacitor_SMD:C_1206_3216Metric_Pad1.33x1.80mm_HandSolder -> Capacitor_SMD:C_0402_1005Metric_Pad0.74x0.62mm_HandSolder
- C3: value 0.47uF -> 1nF; footprint Capacitor_SMD:C_0805_2012Metric_Pad1.18x1.45mm_HandSolder -> Capacitor_SMD:C_0402_1005Metric_Pad0.74x0.62mm_HandSolder
- C4, C5, C6: value C -> 10uF; footprint Capacitor_SMD:C_0805_2012Metric_Pad1.18x1.45mm_HandSolder -> Resistor_SMD:R_2816_7142Metric_Pad3.20x4.45mm_HandSolder
- D1: value D_Zener -> D_Schottky; footprint Diode_SMD:D_SOD-323_HandSoldering -> Diode_SMD:D_SMB-SMC_Universal_Handsoldering
- L01: value 6.8uF -> 15uF; footprint Inductor_SMD:L_10.4x10.4_H4.8 -> Inductor_SMD:L_Coilcraft_XAL1010-XXX
- Q1: value Q_PMOS_GDS -> Si7461DP; footprint Package_SO:TSOP-6_1.65x3.05mm_P0.95mm -> Package_TO_SOT_SMD:TO-263-2
- R1: value 100K -> 255K
- R2: value 0R01 -> 2k210
- R3: footprint Resistor_SMD:R_0805_2012Metric_Pad1.20x1.40mm_HandSolder -> Resistor_SMD:R_1206_3216Metric_Pad1.30x1.75mm_HandSolder
- R4: value - -> 10k
- R5: value 80K6 -> 9K1
- U1: footprint Package_SO:VSSOP-8_3.0x3.0mm_P0.65mm -> Package_SO:VSSOP-8_3x3mm_P0.65mm
- moved Q1 56.3 mm to (41.6, 81.0), turned to 0 degrees
- moved R5 21.9 mm to (106.0, 73.5), turned to 0 degrees
- moved C4 16.8 mm to (91.9, 87.5), turned to 0 degrees
- moved C6 13.2 mm to (91.9, 99.5), turned to 0 degrees
- moved C5 11.7 mm to (91.9, 93.5), turned to 0 degrees
- moved C2 11.2 mm to (107.0, 81.4), turned to -90 degrees
- moved R3 9.04 mm to (105.5, 87.0), turned to 90 degrees
- moved R4 7.52 mm to (101.5, 73.5), turned to 0 degrees
- moved R1 6.02 mm to (101.5, 86.5), turned to 90 degrees
- moved C3 5.57 mm to (103.4, 77.0), turned to 0 degrees
- moved U1 4.42 mm to (103.0, 82.5)
- moved D1 2.48 mm to (95.5, 77.8), turned to 90 degrees
- moved C1 2.14 mm to (100.1, 91.0)
- moved L01 1.53 mm to (86.2, 78.6)
- moved R2 0.68 mm to (103.5, 79.0), turned to 0 degrees
Connections:
- C2 pad 2: GND -> Net-(U1-VCC)
- C3 pad 1: Vin -> Net-(U1-ADJ)
- C3 pad 2: Net-(C3-Pad2) -> Vin
- C4 pad 1: Net-(C4-Pad1) -> Vout (12V)
- C4 pad 2: Vin -> GND
- C5 pad 1: Net-(C5-Pad1) -> Vout (12V)
- C5 pad 2: Net-(C5-Pad2) -> GND
- C6 pad 1: Net-(C5-Pad1) -> Vout (12V)
- C6 pad 2: Vout (12V) -> GND
- D1 pad 1: Net-(Q1-Pad2) -> GND
- D1 pad 2: GND -> Net-(D1-A)
- L01 pad 1: Net-(Q1-Pad2) -> Net-(D1-A)
- L01 pad 2: Net-(C5-Pad1) -> Vout (12V)
- Q1 pad 1: Net-(Q1-Pad2) -> Net-(Q1-G)
- Q1 pad 2: Net-(Q1-Pad2) -> Net-(D1-A)
- Q1 pad 3: Net-(Q1-Pad3) -> Net-(Q1-S)
- R2 pad 1: Net-(C4-Pad1) -> Net-(U1-ADJ)
- R3 pad 2: Net-(Q1-Pad4) -> Net-(Q1-S)
- R4 pad 1: Net-(Q1-Pad2) -> Vout (12V)
- R4 pad 2: Net-(C5-Pad1) -> Net-(U1-FB)
- R5 pad 1: Vout (12V) -> Net-(U1-FB)
- R5 pad 2: Net-(C5-Pad2) -> GND
- U1 pad 1: Net-(C4-Pad1) -> Net-(U1-ADJ)
- U1 pad 3: Net-(C5-Pad2) -> Net-(U1-FB)
- U1 pad 5: Net-(Q1-Pad4) -> Net-(Q1-S)
- U1 pad 6: Net-(Q1-Pad3) -> Net-(Q1-G)
- U1 pad 7: Net-(C3-Pad2) -> Net-(U1-VCC)
Routing:
- net Vin: track 38.4 -> 0.00 mm
- net GND: track 44.8 -> 10.9 mm, vias 2 -> 0
- net Net-(C5-Pad1): track 28.6 -> 0.00 mm
- net Net-(Q1-Pad4): track 19.3 -> 0.00 mm, vias 2 -> 0
- net Net-(U1-RT): track 17.4 -> 0.00 mm
- net Net-(Q1-Pad2): track 15.4 -> 0.00 mm
- net Vout (12V): track 14.6 -> 0.00 mm
- net Net-(C5-Pad2): track 14.4 -> 0.00 mm
- net Net-(C4-Pad1): track 14.4 -> 0.00 mm
- net Net-(Q1-Pad3): track 12.8 -> 0.00 mm, vias 2 -> 0
- net (no net): track 0.00 -> 12.4 mm
- net Net-(C3-Pad2): track 3.67 -> 0.00 mm
- net Net-(R7-Pad1): track 2.54 -> 0.00 mm

Commit message: Update 08/24
Parts:
- removed C5, C6: 10uF, Resistor_SMD:R_2816_7142Metric_Pad3.20x4.45mm_HandSolder
- C1: value 10uF -> 1uF
- C4: footprint Resistor_SMD:R_2816_7142Metric_Pad3.20x4.45mm_HandSolder -> Capacitor_SMD:C_1206_3216Metric_Pad1.33x1.80mm_HandSolder
- D1: footprint Diode_SMD:D_SMB-SMC_Universal_Handsoldering -> Diode_SMD:D_SMB
- L01: value 15uF -> 6.2uF; footprint Inductor_SMD:L_Coilcraft_XAL1010-XXX -> Inductor_SMD:L_Bourns-SRU1028_10.0x10.0mm
- Q1: value Si7461DP -> LM25085; footprint Package_TO_SOT_SMD:TO-263-2 -> Package_SO:TSOP-6_1.65x3.05mm_P0.95mm
- R1: value 255K -> 63k4
- R2: value 2k210 -> 1k430
- R5: value 9K1 -> 1k15
- moved Q1 66.4 mm to (108.0, 77.5)
Connections:
- Q1 pad 1: Net-(Q1-G) -> Net-(D1-A)
- Q1 pad 3: Net-(Q1-S) -> Net-(Q1-G)

Commit message: Update 08/25
Parts:
- moved R5 20.5 mm to (91.0, 87.5)
- moved R4 15.6 mm to (90.0, 84.0)
- moved Q1 6.46 mm to (101.5, 77.8), turned to -90 degrees
- moved C4 4.11 mm to (90.9, 91.5)
- moved C3 4.03 mm to (107.4, 76.5)
- moved R2 4.03 mm to (107.5, 78.5)
- moved L01 1.61 mm to (86.0, 77.0)
- moved D1 0.55 mm to (95.5, 78.3)
Routing:
- net Vout (12V): track 0.00 -> 25.4 mm
- net Vin: track 0.00 -> 25.3 mm
- net Net-(D1-A): track 0.00 -> 20.9 mm
- net Net-(U1-FB): track 0.00 -> 20.8 mm
- net GND: track 10.9 -> 26.0 mm
- net Net-(U1-ADJ): track 0.00 -> 13.9 mm, vias 0 -> 2
- net (no net): track 12.4 -> 0.00 mm
- net Net-(Q1-S): track 0.00 -> 10.1 mm
- net Net-(Q1-G): track 0.00 -> 9.88 mm
- net Net-(U1-RT): track 0.00 -> 4.88 mm
- net Net-(U1-VCC): track 0.00 -> 1.96 mm

Commit message: update 08/25
Other:
- board text added: "CDCR"
Changed lines of the file:
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@@
 		(tags "resistor handsolder")
 		(property "Reference" "R3"
-			(at 0 -1.83 90)
+			(at 0.727064 2.3 90)
 			(layer "F.SilkS")
 			(effects
@@
 		(tags "resistor handsolder")
 		(property "Reference" "R2"
-			(at 0 -1.65 0)
+			(at -0.05 -3.9 0)
 			(layer "F.SilkS")
 			(effects
@@
 		(tags "VSSOP SO JEDEC-MO-187-AA Texas_DGK0008A")
 		(property "Reference" "U1"
-			(at 0 -2.45 0)
+			(at -4.45 1.9 0)
 			(layer "F.SilkS")
 			(effects
@@
 		(tags "Jedec MO-193C TSOP-6L")
 		(property "Reference" "Q1"
-			(at 0 -2.45 90)
+			(at -3.24 -1.78 180)
 			(layer "F.SilkS")
 			(effects
@@
 		(tags "Diode SMB (DO-214AA)")
 		(property "Reference" "D1"
-			(at 0 -3 90)
+			(at 4.3 0.05 180)
 			(layer "F.SilkS")
 			(effects
@@
 		(tags "capacitor handsolder")
 		(property "Reference" "C3"
-			(at 0 -1.16 0)
+			(at 0.0175 -3.5 0)
 			(layer "F.SilkS")
 			(effects
@@
 	(gr_poly
 		(pts
+			(xy 89.75 90.6) (xy 88.45 89) (xy 82 82.75) (xy 82 78.7) (xy 81.4 78.7) (xy 81.4 83.65) (xy 88.45 90.6)
+			(xy 88.45 92.7) (xy 89.75 92.7)
+		)
+		(stroke
+			(width 0.2)
+			(type solid)
+		)
+		(fill yes)
+		(layer "F.Cu")
+		(net 3)
+	)
+	(gr_poly
+		(pts
+			(xy 97.85 91.8) (xy 96.1 91.8) (xy 96.1 91.1) (xy 97.85 91.1)
+		)
+		(stroke
+			(width 0.2)
+			(type solid)
+		)
+		(fill yes)
+		(layer "F.Cu")
+		(net 2)
+	)
+	(gr_poly
+		(pts
+			(xy 100.5 96.45) (xy 100.5 92.5) (xy 103 92.5) (xy 103 96.45)
+		)
+		(stroke
+			(width 0.2)
+			(type solid)
+		)
+		(fill yes)
+		(layer "F.Cu")
+		(net 1)
+	)
+	(gr_poly
+		(pts
+			(xy 87.25 96.45) (xy 87.25 92.5) (xy 89.75 92.5) (xy 89.75 96.45)
+		)
+		(stroke
+			(width 0.2)
+			(type solid)
+		)
+		(fill yes)
+		(layer "F.Cu")
+		(net 3)
+	)
+	(gr_poly
+		(pts
+			(xy 109.5 81.5) (xy 109.5 76) (xy 107.65 76) (xy 107.5 76.2) (xy 107.5 76.8) (xy 107.95 77.35) (xy 107.95 79.95)
+			(xy 107.5 80.35) (xy 106.1 80.35) (xy 105.75 80.75) (xy 105.9 81) (xy 107.95 81) (xy 108 81.5)
+		)
+		(stroke
+			(width 0.2)
+			(type solid)
+		)
+		(fill yes)
+		(layer "F.Cu")
+		(net 1)
+	)
+	(gr_poly
+		(pts
+			(xy 96 96.5) (xy 96 91.05) (xy 92.7 91.05) (xy 92.7 96.5)
+		)
+		(stroke
+			(width 0.2)
+			(type solid)
+		)
+		(fill yes)
+		(layer "F.Cu")
+		(net 2)
+	)
+	(gr_poly
+		(pts
+			(xy 100.5 92.5) (xy 100.5 87) (xy 107 87.05) (xy 108 86) (xy 108 81.5) (xy 109.5 81.5) (xy 109.5 88.5)
+			(xy 107 90.5) (xy 103.5 90.5) (xy 103 91) (xy 103 92.5)
+		)
+		(stroke
+			(width 0.2)
+			(type solid)
+		)
+		(fill yes)
+		(layer "F.Cu")
+		(net 1)
+	)
+	(gr_poly
+		(pts
 			(xy 110 93) (xy 103 93) (xy 103 97) (xy 87 97) (xy 87 93) (xy 80 93) (xy 80 71) (xy 110 71)
 		)
@@
 		(layer "Edge.Cuts")
 	)
+	(gr_text "CDCR"
+		(at 81.1 91.9 0)
+		(layer "F.SilkS")
+		(effects
+			(font
+				(size 1 1)
+				(thickness 0.15)
+			)
+			(justify left bottom)
+		)
+	)
 	(gr_text "Switching node of the PFET must be kept small to avoid radiations, but must be big to dissipate power"
