File: PowerSupply.kicad_pcb (KiCad board)
At the start: 2 copper layers, 30 x 26 mm, 13 parts, among them Q1 LM25085, U1 LM25085

Commit message: update 08-27
Parts:
- moved C1 0.66 mm to (99.4, 91.1)
Changed lines of the file:
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@@
 		(allow_soldermask_bridges_in_footprints no)
 		(tenting front back)
+		(grid_origin 102.35 96.95)
 		(pcbplotparams
 			(layerselection 0x00000000_00000000_55555555_5755f5ff)
@@
 	(footprint "Capacitor_SMD:C_1210_3225Metric_Pad1.33x2.70mm_HandSolder"
 		(layer "F.Cu")
-		(at 100.0625 91 180)
+		(at 99.4125 91.1 180)
 		(descr "Capacitor SMD 1210 (3225 Metric), square (rectangular) end terminal, IPC-7351 nominal with elongated pad for handsoldering. (Body size source: IPC-SM-782 page 76, https://www.pcb-3d.com/wordpress/wp-content/uploads/ipc-sm-782a_amendment_1_and_2.pdf), generated with kicad-footprint-generator")
 		(tags "capacitor handsolder")
@@
 	(gr_poly
 		(pts
-			(xy 100.4 96.765195) (xy 100.4 92.355195) (xy 102.65 92.355195) (xy 102.65 96.765195)
+			(xy 87.35 96.68) (xy 87.35 92.5) (xy 90.77 92.5) (xy 90.77 96.68)
 		)
 		(stroke
 			(width 0)
+			(type solid)
+		)
+		(fill yes)
+		(layer "F.Cu")
+		(net 3)
+	)
+	(gr_poly
+		(pts
+			(xy 109.5 81.5) (xy 109.5 76) (xy 107.73 76) (xy 107.73 76) (xy 107.73 77.081112) (xy 107.95 77.35)
+			(xy 107.95 79.95) (xy 107.5 80.35) (xy 106.1 80.35) (xy 105.75 80.75) (xy 105.9 81) (xy 107.95 81)
+			(xy 108 81.5)
+		)
+		(stroke
+			(width 0.2)
 			(type solid)
 		)
@@
 	(gr_poly
 		(pts
-			(xy 87.25 96.78) (xy 87.25 92.5) (xy 90.77 92.5) (xy 90.77 96.78)
+			(xy 102.8 96.8) (xy 102.8 92.1) (xy 100.35 92.1) (xy 100.35 96.8)
 		)
 		(stroke
 			(width 0)
-			(type solid)
-		)
-		(fill yes)
-		(layer "F.Cu")
-		(net 3)
-	)
-	(gr_poly
-		(pts
-			(xy 109.5 81.5) (xy 109.5 76) (xy 107.65 76) (xy 107.5 76.2) (xy 107.5 76.8) (xy 107.95 77.35) (xy 107.95 79.95)
-			(xy 107.5 80.35) (xy 106.1 80.35) (xy 105.75 80.75) (xy 105.9 81) (xy 107.95 81) (xy 108 81.5)
-		)
-		(stroke
-			(width 0.2)
 			(type solid)
 		)
@@
 	(gr_poly
 		(pts
-			(xy 98.6416 96.78) (xy 98.6416 85.58) (xy 91.86 85.58) (xy 91.86 96.78)
+			(xy 98.6416 96.68) (xy 98.6416 85.58) (xy 91.86 85.58) (xy 91.86 96.68)
 		)
 		(stroke
@@
 	(gr_poly
 		(pts
-			(xy 100.5 92.5) (xy 100.5 87) (xy 107 87.05) (xy 108 86) (xy 108 81.5) (xy 109.5 81.5) (xy 109.5 88.5)
-			(xy 107 90.5) (xy 103.5 90.5) (xy 103 91) (xy 103 92.5)
+			(xy 100.43 92.25) (xy 100.44 87) (xy 106.94 87.05) (xy 107.94 86) (xy 107.94 81.5) (xy 109.44 81.5)
+			(xy 109.44 88.5) (xy 106.94 90.5) (xy 105.03 90.5) (xy 102.6 92.25)
 		)
 		(stroke
@@
 	(dimension
 		(type orthogonal)
-		(layer "B.SilkS")
+		(layer "User.1")
 		(pts
 			(xy 91.86 95.49) (xy 98.64 95.45)
@@
 		(gr_text "6.7800 mm"
 			(at 95.25 103 0)
-			(layer "B.SilkS")
+			(layer "User.1")
 			(effects
 				(font
@@
 	(dimension
 		(type orthogonal)
-		(layer "B.SilkS")
+		(layer "User.1")
 		(pts
 			(xy 87.25 96.45) (xy 90.77 96.45)
@@
 		(gr_text "3.5200 mm"
 			(at 89.01 97.46 0)
-			(layer "B.SilkS")
+			(layer "User.1")
 			(effects
 				(font
@@
 	(dimension
 		(type orthogonal)
-		(layer "B.SilkS")
+		(layer "User.1")
 		(pts
 			(xy 90.77 95.26) (xy 91.86 95.49)
@@
 		(gr_text "1.0900 mm"
 			(at 91.315 100.03 0)
-			(layer "B.SilkS")
-			(effects
-				(font
+			(layer "User.1")
+			(effects
+				(font

Commit message: Update 08-27
Parts:
- moved Q1 0.84 mm to (102.4, 78.0), turned to 0 degrees
Routing:
- net Net-(Q1-S): track 10.1 -> 17.5 mm, vias 0 -> 2
- net Net-(U1-ADJ): track 13.9 -> 15.6 mm
- net Net-(D1-A): track 20.9 -> 21.8 mm
- net Net-(Q1-G): track 9.88 -> 10.7 mm, vias 0 -> 2
- net GND: vias 0 -> 6
- added copper zone on B.Cu, net GND
- added copper zone on F.Cu, net GND
Other:
- board text added: "GND"
- board text added: "Vin"
- board text added: "Vout"
- board text removed: "Switching node of the PFET must be kept small to avoid radiations, but must be big to dissipate power"

Commit message: Update 27-08
Parts:
- moved C4 1.52 mm to (90.9, 90.0)
- moved C2 0.94 mm to (107.6, 82.1), turned to 180 degrees
- moved C1 0.52 mm to (99.4, 90.6)
Routing:
- net Vin: track 25.3 -> 24.3 mm
- net GND: track 26.0 -> 25.3 mm
Other:
- board text added: "JLCJLCJLCJLC"

Commit message: Update 08-28
Parts:
- Q1: value LM25085 -> SQ3419AEEV
- R2: value 1k430 -> 1k4
- U1: footprint Package_SO:VSSOP-8_3x3mm_P0.65mm -> Package_SO:HVSSOP-8-1EP_3x3mm_P0.65mm_EP1.57x1.89mm_ThermalVias
- moved R1 8.09 mm to (103.2, 78.6), turned to 180 degrees
- moved Q1 2.66 mm to (102.6, 75.4)
Routing:
- net Net-(Q1-G): track 10.7 -> 18.1 mm
- net Net-(Q1-S): track 17.5 -> 24.2 mm
- net Net-(U1-ADJ): track 15.6 -> 10.5 mm, vias 2 -> 0
- net Vin: track 24.3 -> 29.3 mm
- net Net-(U1-RT): track 4.88 -> 7.88 mm
- net Net-(D1-A): track 21.8 -> 21.3 mm

Commit message: Update 08-28
Parts:
- D1: footprint Diode_SMD:D_SMB -> Diode_SMD:D_SMC
Routing:
- net GND: track 25.3 -> 23.9 mm

Commit message: Final Layout
Routing:
- net Vin: track 29.3 -> 34.4 mm, vias 0 -> 4
- net Vout (12V): track 25.4 -> 30.5 mm, vias 0 -> 4
