File: PowerSupply.kicad_sch (KiCad schematic)
At the start: 13 parts, among them Q1 SQ3419AEEV, U1 LM25085

Commit message: Final Layout
Parts:
- C4: symbol Device:C -> Device:C_Polarized_US
Changed lines of the file:
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@@
 	)
 	(symbol
-		(lib_id "Device:C")
+		(lib_id "Device:C_Polarized_US")
 		(at 175.26 114.3 0)
 		(unit 1)
@@
 		(fields_autoplaced yes)
 		(property "Reference" "C4"
-			(at 179.07 113.0299 0)
+			(at 179.07 112.3949 0)
 			(effects
 				(font
@@
 		)
 		(property "Value" "10uF"
-			(at 179.07 115.5699 0)
+			(at 179.07 114.9349 0)
 			(effects
 				(font
@@
 		)
 		(property "Footprint" "Capacitor_SMD:C_1206_3216Metric_Pad1.33x1.80mm_HandSolder"
-			(at 176.2252 118.11 0)
+			(at 175.26 114.3 0)
 			(effects
 				(font
@@
 			)
 		)
-		(property "Description" ""
+		(property "Description" "Polarized capacitor, US symbol"
 			(at 175.26 114.3 0)
 			(effects
